Commit message: feat: add cox, femur urdf

File: robots/hexapod.urdf.xacro (robot description, xacro)
@@ -1,3 +1,26 @@
 <?xml version="1.0"?>
-<robot xmlns:xacro="http://www.ros.org/wiki/xacro">
+<robot name="hexapod" xmlns:xacro="http://www.ros.org/wiki/xacro">
+    <xacro:include filename="$(find hexapod)/urdf/general.urdf.xacro"/>
+    <xacro:include filename="$(find hexapod)/urdf/body.urdf.xacro"/>
+    <xacro:include filename="$(find hexapod)/urdf/cox.urdf.xacro"/>
+    <xacro:include filename="$(find hexapod)/urdf/femur.urdf.xacro"/>
+    <!-- <xacro:include filename="$(find hexapod)/urdf/hexapod.gazebo" /> -->
+    <!-- Footprint link -->
+    <link name="base_footprint">
+        <visual>
+            <geometry>
+                <cylinder length="0.001" radius="0.01"/>
+            </geometry>
+        </visual>
+    </link>
+    <!-- Floating-base Joint -->
+    <!-- <joint name="floating_base" type="fixed">
+        <origin xyz="0 0 0" rpy="0 0 0"/>
+        <parent link="base_footprint"/>
+        <child link="heaxpod_body_link"/>
+    </joint> -->
+    <!-- <xacro:generate_body/> -->
+    <xacro:generate_body/>
+    <xacro:generate_cox side="left"/>
+    <xacro:generate_femur side="left"/>
 </robot>

File: urdf/general.urdf.xacro (robot description, xacro)
@@ -1,12 +1,13 @@
 <?xml version="1.0"?>
 <robot xmlns:xacro="http://www.ros.org/wiki/xacro">
-    <xacro:property name="DOCK_IXX" value="0.00531683333333"/>
-    <xacro:property name="DOCK_IYY" value="0.00531683333333"/>
-    <xacro:property name="DOCK_IZZ" value="0.010143"/>
+    <xacro:property name="HEX_IXX" value="0.00531683333333"/>
+    <xacro:property name="HEX_IYY" value="0.00531683333333"/>
+    <xacro:property name="HEX_IZZ" value="0.010143"/>
 <!--Physical properties of material-->
-    <xacro:property name="DOCK_MU1" value="10.0"/>  <!-- Frictions -->
-    <xacro:property name="DOCK_MU2" value="10.0"/>
-    <xacro:property name="DOCK_KP" value="10000.0"/> <!-- Static contact stiffness. This determines if the link material is closer to marble (very rigid, bigger values) or more like rubber (soft material, lower values). -->
-    <xacro:property name="DOCK_KD" value="10000.0"/> <!-- Dynamic contact stiffness. This determines if the link material is closer to marble (very rigid, bigger values) or more like rubber (soft material, lower values). It's essentially how much it deforms over a long period of time, exerting its pressure. -->
+    <xacro:property name="HEX_MU1" value="10.0"/>  <!-- Frictions -->
+    <xacro:property name="HEX_MU2" value="10.0"/>
+    <xacro:property name="HEX_KP" value="10000.0"/> <!-- Static contact stiffness. This determines if the link material is closer to marble (very rigid, bigger values) or more like rubber (soft material, lower values). -->
+    <xacro:property name="HEX_KD" value="10000.0"/> <!-- Dynamic contact stiffness. This determines if the link material is closer to marble (very rigid, bigger values) or more like rubber (soft material, lower values). It's essentially how much it deforms over a long period of time, exerting its pressure. -->
+    <xacro:property name="SCALE" value="0.001"/>
 <!-- ################################################################## -->
 <!-- ############################ MATH ################################ -->
@@ -34,4 +35,10 @@
                 <sphere radius="${radius}"/>
             </xacro:if>
+        </geometry>
+    </xacro:macro>
+<!--########################## STL XACRO ##########################-->
+    <xacro:macro name="add_stl" params="scale fname">
+        <geometry>
+            <mesh filename="package://hexapod/urdf/models/${fname}.stl" scale="${scale} ${scale} ${scale}"/>
         </geometry>
     </xacro:macro>

Commit message: feat: made YAML/macros for assigning joint origins

File: robots/hexapod.urdf.xacro (robot description, xacro)
@@ -21,4 +21,6 @@
     <!-- <xacro:generate_body/> -->
     <xacro:generate_body/>
-    <xacro:generate_leg side="left"/>
+    <xacro:generate_leg side="R" position="M"/>
+    <xacro:generate_leg side="R" position="F"/>
+    <xacro:generate_leg side="R" position="B"/>
 </robot>

File: urdf/body.urdf.xacro (robot description, xacro)
@@ -16,8 +16,8 @@
         <link name="body_link">
             <collision>
-                <xacro:add_stl scale="${SCALE}" fname="baseWithCox"/>
+                <xacro:add_stl scale="${SCALE}" fname="base"/>
             </collision>
             <visual>
-                <xacro:add_stl scale="${SCALE}" fname="baseWithCox"/>
+                <xacro:add_stl scale="${SCALE}" fname="base"/>
             </visual>
             <xacro:MINIMUM_INERTIAL/>

File: urdf/cox.urdf.xacro (robot description, xacro)
@@ -1,39 +1,18 @@
 <?xml version="1.0"?>
 <robot xmlns:xacro="http://www.ros.org/wiki/xacro">
-    <!-- <xacro:property name="DOCK_MASS" value="0.01"/> -->
-    <xacro:property name="COX_WJ_X" value="-0.0635"/> <!-- 063501 -->
-    <xacro:property name="COX_WJ_Y" value="0.0"/>
-    <xacro:property name="COX_WJ_Z" value="0.003"/>
-    <xacro:property name="TROCOX_X" value="-0.063406"/>
-    <xacro:property name="TROCOX_Y" value="-0.069967"/>
-    <xacro:property name="TROCOX_Z" value="0.023007"/>
-    <xacro:macro name="COX_MOTOR_WHEEL_JOINT_ORIGIN">
-        <origin xyz="${COX_WJ_X} ${COX_WJ_Y} ${COX_WJ_Z}" rpy="${PI_2} ${PI} 0" />
-    </xacro:macro>
-    <xacro:macro name="TROCOX_JOINT_ORIGIN">
-        <!-- <origin xyz="${TROCOX_X} ${TROCOX_Y} ${TROCOX_Z}" rpy="0 0 0" /> -->
-        <origin xyz="0 0 0" rpy="${PI} 0 0" />
-    </xacro:macro>
-<!-- ########################## HEXAPOD LEG GENERATOR ############################ -->
-    <xacro:macro name="generate_cox" params="side">
-        <link name="cox_motor_wheel_link">
-            <collision>
-                <xacro:add_stl scale="${SCALE}" fname="ax12_wheel_faceOrigin"/>
-            </collision>
-            <visual>
-                <xacro:add_stl scale="${SCALE}" fname="ax12_wheel_faceOrigin"/>
-            </visual>
-            <xacro:MINIMUM_INERTIAL/>
-        </link>
-        <joint name="cox_motor_wheel_joint" type="revolute" >
-            <xacro:COX_MOTOR_WHEEL_JOINT_ORIGIN/>
+<!-- ########################## HEXAPOD TROCOX GENERATOR ############################ -->
+    <xacro:macro name="generate_cox" params="side position joint_type:=COX">
+        <xacro:generate_IdOr_link_same_mesh link_name="${side}_${position}_COX_link" stl="coxa_2_wheels_${position}_fo"/>
+        <xacro:property name="coords" value="${origins[side][position][joint_type]}"/>
+        <joint name="${side}_${position}_COX_joint" type="revolute" >
+            <origin xyz="${coords['x']} ${coords['y']} ${coords['z']}" rpy="0 0 0"/>
             <parent link="body_link"/>
-            <child link="cox_motor_wheel_link"/>
-            <axis xyz="0 1 0" rpy="0 0 0"/>
+            <child link="${side}_${position}_COX_link"/>
+            <axis xyz="0 0 1" rpy="0 0 0"/>
             <!-- <limit upper="${PI}" lower="${PI}" effort="10000" velocity="1000"/> -->
             <limit upper="1.0" lower="-1.0" effort="1000.0" velocity="0.5"/>
             <!-- <joint_properties damping="1.0" friction="1.0"/> -->
         </joint>
-         <gazebo reference="cox_motor_wheel_link">
+         <gazebo reference="${side}_${position}_COX_link">
              <mu1 value="${HEX_MU1}"/>
              <mu2 value="${HEX_MU2}"/>
@@ -41,30 +20,4 @@
              <kd value="${HEX_KD}"/>
               <material>Gazebo/Green</material>
-        </gazebo>
-<!-- ########################## TROCOX ############################ -->
-        <link name="trocox_link">
-            <collision>
-                <xacro:add_stl scale="${SCALE}" fname="trochanter_contactOrigin"/>
-            </collision>
-            <visual>
-                <xacro:add_stl scale="${SCALE}" fname="trochanter_contactOrigin"/>
-            </visual>
-            <xacro:MINIMUM_INERTIAL/>
-        </link>
-        <joint name="trocox_joint" type="fixed" >
-            <xacro:TROCOX_JOINT_ORIGIN/>
-            <parent link="cox_motor_wheel_link"/>
-            <child link="trocox_link"/>
-            <!-- <axis xyz="0 0 1" rpy="0 0 0"/> -->
-            <!-- <limit upper="${PI}" lower="${PI}" effort="10000" velocity="1000"/> -->
-            <!-- <limit upper="1.0" lower="-1.0" effort="1000.0" velocity="0.5"/> -->
-            <!-- <joint_properties damping="1.0" friction="1.0"/> -->
-        </joint>
-         <gazebo reference="trocox_link">
-             <mu1 value="${HEX_MU1}"/>
-             <mu2 value="${HEX_MU2}"/>
-             <kp value="${HEX_KP}"/>
-             <kd value="${HEX_KD}"/>
-              <material>Gazebo/Red</material>
         </gazebo>
         <!-- <transmission name="${side}_dock_transmission">

File: urdf/femur.urdf.xacro (robot description, xacro)
@@ -1,41 +1,12 @@
 <?xml version="1.0"?>
 <robot xmlns:xacro="http://www.ros.org/wiki/xacro">
-    <!-- <xacro:property name="DOCK_MASS" value="0.01"/> -->
-    <xacro:property name="FEM_WJ_X" value="-0.070807"/>
-    <xacro:property name="FEM_WJ_Y" value="0.02"/>
-    <xacro:property name="FEM_WJ_Z" value="0.064307"/>
-    <!-- FROM ORIGIN -->
-    <xacro:macro name="FEM_MOTOR_WHEEL_JOINT_ORIGIN">
-        <origin xyz="${FEM_WJ_X} ${FEM_WJ_Y} ${FEM_WJ_Z}" rpy="${PI_2} ${PI} 0" />
-    </xacro:macro>
-    <xacro:property name="FEM_WJ_TCX_OFFSET_X" value="0.007307"/>
-    <xacro:property name="FEM_WJ_TCX_OFFSET_Y" value="0.061307"/>
-    <xacro:property name="FEM_WJ_TCX_OFFSET_Z" value="-0.02"/>
-    <!-- FROM TROCOX JOINT -->
-    <xacro:macro name="FEM_MOTOR_WHEEL_JOINT_ORIGIN_TCX_OFFSET">
-        <origin xyz="${FEM_WJ_TCX_OFFSET_X} ${FEM_WJ_TCX_OFFSET_Y} ${FEM_WJ_TCX_OFFSET_Z} " rpy="-${PI_2} 0 -${PI_2}" />
-    </xacro:macro>
-    <!-- FROM TROCOX JOINT -->
-    <xacro:macro name="FEMUR_JOINT_ORIGIN_TCX_OFFSET">
-        <origin xyz="0 -0.004 0" rpy="0 -${PI_2} 0" />
-    </xacro:macro>
-<!-- ########################## HEXAPOD LEG GENERATOR ############################ -->
-    <xacro:macro name="generate_femur" params="side">
-<!-- ########################## FEM WHEEL ############################ -->
-        <link name="fem_motor_wheel_link">
-            <xacro:FEM_MOTOR_WHEEL_JOINT_ORIGIN_TCX_OFFSET/>
-            <collision>
-                <xacro:add_stl scale="${SCALE}" fname="ax12_wheel_faceOrigin"/>
-            </collision>
-            <visual>
-                <xacro:add_stl scale="${SCALE}" fname="ax12_wheel_faceOrigin"/>
-            </visual>
-            <xacro:MINIMUM_INERTIAL/>
-        </link>
-        <joint name="fem_motor_wheel_joint" type="revolute" >
-            <!-- <xacro:FEM_MOTOR_WHEEL_JOINT_ORIGIN/> -->
-            <xacro:FEM_MOTOR_WHEEL_JOINT_ORIGIN_TCX_OFFSET/>
-            <parent link="trocox_link"/>
-            <child link="fem_motor_wheel_link"/>
+<!-- ########################## HEXAPOD FEMUR GENERATOR ############################ -->
+    <xacro:macro name="generate_femur" params="side position joint_type:=FEM">
+        <xacro:generate_IdOr_link_same_mesh link_name="${side}_${position}_FEM_link" stl="femur_no_wheel_${position}_fo"/>
+        <xacro:property name="coords" value="${origins[side][position][joint_type]}"/>
+        <joint name="${side}_${position}_FEM_joint" type="revolute" >
+            <origin xyz="${coords['x']} ${coords['y']} ${coords['z']}" rpy="0 0 0"/>
+            <parent link="${side}_${position}_COX_link"/>
+            <child link="${side}_${position}_FEM_link"/>
             <axis xyz="0 1 0" rpy="0 0 0"/>
             <!-- <limit upper="${PI}" lower="${PI}" effort="10000" velocity="1000"/> -->
@@ -43,27 +14,5 @@
             <!-- <joint_properties damping="1.0" friction="1.0"/> -->
         </joint>
-         <gazebo reference="fem_motor_wheel_link">
-             <mu1 value="${HEX_MU1}"/>
-             <mu2 value="${HEX_MU2}"/>
-             <kp value="${HEX_KP}"/>
-             <kd value="${HEX_KD}"/>
-              <material>Gazebo/Blue</material>
-        </gazebo>
-<!-- ########################## FEMUR ############################ -->
-        <link name="femur_link">
-            <collision>
-                <xacro:add_stl scale="${SCALE}" fname="femur_pPls"/>
-            </collision>
-            <visual>
-                <xacro:add_stl scale="${SCALE}" fname="femur_pPls"/>
-            </visual>
-            <xacro:MINIMUM_INERTIAL/>
-        </link>
-        <joint name="femur_joint" type="fixed" >
-            <xacro:FEMUR_JOINT_ORIGIN_TCX_OFFSET/>
-            <parent link="fem_motor_wheel_link"/>
-            <child link="femur_link"/>
-        </joint>
-         <gazebo reference="fem_motor_wheel_link">
+         <gazebo reference="${side}_${position}_FEM_link">
              <mu1 value="${HEX_MU1}"/>
              <mu2 value="${HEX_MU2}"/>

File: urdf/general.urdf.xacro (robot description, xacro)
@@ -37,4 +37,28 @@
         </geometry>
     </xacro:macro>
+<!--########################## GENERATE IDENTITY ORIGIN LINK WITH IDENTICAL COLLISION/VISUAL MESH XACRO ##########################-->
+    <xacro:macro name="generate_IdOr_link_same_mesh" params="link_name stl">
+        <link name="${link_name}">
+            <collision>
+                <xacro:add_stl scale="${SCALE}" fname="${stl}"/>
+            </collision>
+            <visual>
+                <xacro:add_stl scale="${SCALE}" fname="${stl}"/>
+            </visual>
+            <xacro:MINIMUM_INERTIAL/>
+        </link>
+    </xacro:macro>
+    <!--########################## GENERATE IDENTITY ORIGIN LINK WITH IDENTICAL COLLISION/VISUAL MESH XACRO ##########################-->
+    <!-- <xacro:macro name="generate_joint" params="joint_name parent child ">
+        <link name="${link_name}">
+            <collision>
+                <xacro:add_stl scale="${SCALE}" fname="${stl}"/>
+            </collision>
+            <visual>
+                <xacro:add_stl scale="${SCALE}" fname="${stl}"/>
+            </visual>
+            <xacro:MINIMUM_INERTIAL/>
+        </link>
+    </xacro:macro> -->
 <!--########################## STL XACRO ##########################-->
     <xacro:macro name="add_stl" params="scale fname">

File: urdf/leg.urdf.xacro (robot description, xacro)
@@ -1,13 +1,14 @@
 <?xml version="1.0"?>
-<robot name="hexapod" xmlns:xacro="http://www.ros.org/wiki/xacro">
+<robot xmlns:xacro="http://www.ros.org/wiki/xacro">
     <!-- <xacro:include filename="$(find hexapod)/urdf/general.urdf.xacro"/> -->
+    <xacro:include filename="$(find hexapod)/urdf/joint_origins.urdf.xacro"/>
     <xacro:include filename="$(find hexapod)/urdf/cox.urdf.xacro"/>
     <xacro:include filename="$(find hexapod)/urdf/femur.urdf.xacro"/>
     <xacro:include filename="$(find hexapod)/urdf/tibia.urdf.xacro"/>
 <!-- ########################## HEXAPOD LEG GENERATOR ############################ -->
-    <xacro:macro name="generate_leg" params="side">
-        <xacro:generate_cox side="left"/>
-        <xacro:generate_femur side="left"/>
-        <xacro:generate_tibia side="left"/>
+    <xacro:macro name="generate_leg" params="side position">
+        <xacro:generate_cox side="${side}" position="${position}"/>
+        <xacro:generate_femur side="${side}" position="${position}"/>
+        <!-- <xacro:generate_tibia side="left"/> -->
     </xacro:macro>
 <!-- ########################## END HEXAPOD LEG GENERATOR ############################ -->
