Commit message: refactor: setup new xacro for leg generation

File: robots/hexapod.urdf (robot description, URDF)
Before this commit: robot hexapod, 3 links, 2 joints
Links:
- added link fem_motor_wheel_link, mass 0.1; collision mesh filename=package://hexapod/urdf/models/ax12_wheel_faceOrigin.stl scale=0.001 0.001 0.001; visual mesh filename=package://hexapod/urdf/models/ax12_wheel_faceOrigin.stl scale=0.001 0.001 0.001
- added link femur_link, mass 0.1; collision mesh filename=package://hexapod/urdf/models/femur_pPls.stl scale=0.001 0.001 0.001; visual mesh filename=package://hexapod/urdf/models/femur_pPls.stl scale=0.001 0.001 0.001
- added link tib_motor_wheel_link, mass 0.1; collision mesh filename=package://hexapod/urdf/models/ax12_wheel_faceOrigin.stl scale=0.001 0.001 0.001; visual mesh filename=package://hexapod/urdf/models/ax12_wheel_faceOrigin.stl scale=0.001 0.001 0.001
- added link tibia_link, mass 0.1; collision mesh filename=package://hexapod/urdf/models/tib3piece_centered.stl scale=0.001 0.001 0.001; visual mesh filename=package://hexapod/urdf/models/tib3piece_centered.stl scale=0.001 0.001 0.001
- added link trocox_link, mass 0.1; collision mesh filename=package://hexapod/urdf/models/trochanter_contactOrigin.stl scale=0.001 0.001 0.001; visual mesh filename=package://hexapod/urdf/models/trochanter_contactOrigin.stl scale=0.001 0.001 0.001
- link cox_motor_wheel_link: geometry collision mesh filename=package://hexapod/urdf/models/ax12_wheel_faceOrigin.stl scale=0.001 0.001 0.001; visual mesh filename=package://hexapod/urdf/models/ax12_wheel_faceOrigin.stl scale=0.001 0.001 0.001
Joints:
- added joint fem_motor_wheel_joint: type revolute, parent trocox_link, child fem_motor_wheel_link, origin xyz=0.007307 0.061307 -0.02  rpy=-1.57079632679 0 -1.57079632679, axis 0 1 0, limit lower=-1.0 upper=1.0 effort=1000.0 velocity=0.5
- added joint femur_joint: type fixed, parent fem_motor_wheel_link, child femur_link, origin xyz=0 -0.004 0 rpy=0 -1.57079632679 0
- added joint tib_motor_wheel_joint: type revolute, parent femur_link, child tib_motor_wheel_link, origin xyz=0.032 0.004 0.0  rpy=0 0 0, axis 0 1 0, limit lower=-1.0 upper=1.0 effort=1000.0 velocity=0.5
- added joint tibia_joint: type fixed, parent tib_motor_wheel_link, child tibia_link, origin xyz=0.0 -0.019924 -0.01826 rpy=0 0 -3.14
- added joint trocox_joint: type fixed, parent cox_motor_wheel_link, child trocox_link, origin xyz=0 0 0 rpy=3.14 0 0
- joint cox_motor_wheel_joint: axis 0 0 1 -> 0 1 0; limit (none) -> lower=-1.0 upper=1.0 effort=1000.0 velocity=0.5; origin xyz=-0.0635 0.0 0.005 rpy=1.57 0 0 -> xyz=-0.0635 0.0 0.003 rpy=1.57079632679 3.14 0

File: robots/hexapod.urdf.xacro (robot description, xacro)
@@ -3,7 +3,5 @@
     <xacro:include filename="$(find hexapod)/urdf/general.urdf.xacro"/>
     <xacro:include filename="$(find hexapod)/urdf/body.urdf.xacro"/>
-    <xacro:include filename="$(find hexapod)/urdf/cox.urdf.xacro"/>
-    <xacro:include filename="$(find hexapod)/urdf/femur.urdf.xacro"/>
-    <xacro:include filename="$(find hexapod)/urdf/tibia.urdf.xacro"/>
+    <xacro:include filename="$(find hexapod)/urdf/leg.urdf.xacro"/>
     <!-- <xacro:include filename="$(find hexapod)/urdf/hexapod.gazebo" /> -->
     <!-- Footprint link -->
@@ -23,6 +21,4 @@
     <!-- <xacro:generate_body/> -->
     <xacro:generate_body/>
-    <xacro:generate_cox side="left"/>
-    <xacro:generate_femur side="left"/>
-    <xacro:generate_tibia side="left"/>
+    <xacro:generate_leg side="left"/>
 </robot>

File: urdf/tibia.urdf.xacro (robot description, xacro)
@@ -27,5 +27,5 @@
         <origin xyz="${TIB_FEM_OFFSET_X} ${TIB_FEM_OFFSET_Y} ${TIB_FEM_OFFSET_Z}" rpy="0 0 -${PI}" />
     </xacro:macro>
-<!-- ########################## HEXAPOD LEG GENERATOR ############################ -->
+<!-- ########################## HEXAPOD TIBIA GENERATOR ############################ -->
     <xacro:macro name="generate_tibia" params="side">
 <!-- ########################## FEM WHEEL ############################ -->

Commit message: work on IKfast and MoveIt tutorials.

File: robots/hexapod.urdf (robot description, URDF)
Before this commit: robot hexapod, 8 links, 7 joints
Links:
- added link L_B_COX_link, mass 0.1; collision mesh filename=package://hexapod/urdf/models/coxa_L_B.stl scale=0.001 0.001 0.001; visual mesh filename=package://hexapod/urdf/models/coxa_L_B.stl scale=0.001 0.001 0.001
- added link L_B_FEM_link, mass 0.1; collision mesh filename=package://hexapod/urdf/models/femur_L_B.stl scale=0.001 0.001 0.001; visual mesh filename=package://hexapod/urdf/models/femur_L_B.stl scale=0.001 0.001 0.001
- added link L_B_TIB_link, mass 0.1; collision mesh filename=package://hexapod/urdf/models/tibia_L_B.stl scale=0.001 0.001 0.001; visual mesh filename=package://hexapod/urdf/models/tibia_L_B.stl scale=0.001 0.001 0.001
- added link L_F_COX_link, mass 0.1; collision mesh filename=package://hexapod/urdf/models/coxa_L_F.stl scale=0.001 0.001 0.001; visual mesh filename=package://hexapod/urdf/models/coxa_L_F.stl scale=0.001 0.001 0.001
- added link L_F_FEM_link, mass 0.1; collision mesh filename=package://hexapod/urdf/models/femur_L_F.stl scale=0.001 0.001 0.001; visual mesh filename=package://hexapod/urdf/models/femur_L_F.stl scale=0.001 0.001 0.001
- added link L_F_TIB_link, mass 0.1; collision mesh filename=package://hexapod/urdf/models/tibia_L_F.stl scale=0.001 0.001 0.001; visual mesh filename=package://hexapod/urdf/models/tibia_L_F.stl scale=0.001 0.001 0.001
- added link L_M_COX_link, mass 0.1; collision mesh filename=package://hexapod/urdf/models/coxa_L_M.stl scale=0.001 0.001 0.001; visual mesh filename=package://hexapod/urdf/models/coxa_L_M.stl scale=0.001 0.001 0.001
- added link L_M_FEM_link, mass 0.1; collision mesh filename=package://hexapod/urdf/models/femur_L_M.stl scale=0.001 0.001 0.001; visual mesh filename=package://hexapod/urdf/models/femur_L_M.stl scale=0.001 0.001 0.001
- added link L_M_TIB_link, mass 0.1; collision mesh filename=package://hexapod/urdf/models/tibia_L_M.stl scale=0.001 0.001 0.001; visual mesh filename=package://hexapod/urdf/models/tibia_L_M.stl scale=0.001 0.001 0.001
- added link R_B_TIB_link, mass 0.1; collision mesh filename=package://hexapod/urdf/models/tibia_R_B.stl scale=0.001 0.001 0.001; visual mesh filename=package://hexapod/urdf/models/tibia_R_B.stl scale=0.001 0.001 0.001
- added link R_F_TIB_link, mass 0.1; collision mesh filename=package://hexapod/urdf/models/tibia_R_F.stl scale=0.001 0.001 0.001; visual mesh filename=package://hexapod/urdf/models/tibia_R_F.stl scale=0.001 0.001 0.001
- added link R_M_TIB_link, mass 0.1; collision mesh filename=package://hexapod/urdf/models/tibia_R_M.stl scale=0.001 0.001 0.001; visual mesh filename=package://hexapod/urdf/models/tibia_R_M.stl scale=0.001 0.001 0.001
- link R_B_COX_link: geometry collision mesh filename=package://hexapod/urdf/models/coxa_R_B.stl scale=0.001 0.001 0.001; visual mesh filename=package://hexapod/urdf/models/coxa_R_B.stl scale=0.001 0.001 0.001
- link R_B_FEM_link: geometry collision mesh filename=package://hexapod/urdf/models/femur_R_B.stl scale=0.001 0.001 0.001; visual mesh filename=package://hexapod/urdf/models/femur_R_B.stl scale=0.001 0.001 0.001
- link R_F_COX_link: geometry collision mesh filename=package://hexapod/urdf/models/coxa_R_F.stl scale=0.001 0.001 0.001; visual mesh filename=package://hexapod/urdf/models/coxa_R_F.stl scale=0.001 0.001 0.001
- link R_F_FEM_link: geometry collision mesh filename=package://hexapod/urdf/models/femur_R_F.stl scale=0.001 0.001 0.001; visual mesh filename=package://hexapod/urdf/models/femur_R_F.stl scale=0.001 0.001 0.001
- link R_M_COX_link: geometry collision mesh filename=package://hexapod/urdf/models/coxa_R_M.stl scale=0.001 0.001 0.001; visual mesh filename=package://hexapod/urdf/models/coxa_R_M.stl scale=0.001 0.001 0.001
- link R_M_FEM_link: geometry collision mesh filename=package://hexapod/urdf/models/femur_R_M.stl scale=0.001 0.001 0.001; visual mesh filename=package://hexapod/urdf/models/femur_R_M.stl scale=0.001 0.001 0.001
Joints:
- added joint L_B_COX_joint: type revolute, parent body_link, child L_B_COX_link, origin xyz=0.057077 0.066312 0.007 rpy=0 0 0, axis 0 0 1, limit lower=-1.0 upper=1.0 effort=1000.0 velocity=0.5
- added joint L_B_FEM_joint: type revolute, parent L_B_COX_link, child L_B_FEM_link, origin xyz=0.007261 0.017438 0.057284 rpy=0 0 0, axis 0 1 0, limit lower=-1.0 upper=1.0 effort=1000.0 velocity=0.5
- added joint L_B_TIB_joint: type revolute, parent L_B_FEM_link, child L_B_TIB_link, origin xyz=0.027712 0 0 rpy=0 0 0, axis 0 1 0, limit lower=-1.0 upper=1.0 effort=1000.0 velocity=0.5
- added joint L_F_COX_joint: type revolute, parent body_link, child L_F_COX_link, origin xyz=0.057077 -0.066312 0.007 rpy=0 0 0, axis 0 0 1, limit lower=-1.0 upper=1.0 effort=1000.0 velocity=0.5
- added joint L_F_FEM_joint: type revolute, parent L_F_COX_link, child L_F_FEM_link, origin xyz=0.007261 -0.017448 0.057284 rpy=0 0 0, axis 0 1 0, limit lower=-1.0 upper=1.0 effort=1000.0 velocity=0.5
- added joint L_F_TIB_joint: type revolute, parent L_F_FEM_link, child L_F_TIB_link, origin xyz=0.027712 0 0 rpy=0 0 0, axis 0 1 0, limit lower=-1.0 upper=1.0 effort=1000.0 velocity=0.5
- added joint L_M_COX_joint: type revolute, parent body_link, child L_M_COX_link, origin xyz=0.0635 0 0.007 rpy=0 0 0, axis 0 0 1, limit lower=-1.0 upper=1.0 effort=1000.0 velocity=0.5
- added joint L_M_FEM_joint: type revolute, parent L_M_COX_link, child L_M_FEM_link, origin xyz=0.007261 0.015954 0.057284 rpy=0 0 0, axis 0 1 0, limit lower=-1.0 upper=1.0 effort=1000.0 velocity=0.5
- added joint L_M_TIB_joint: type revolute, parent L_M_FEM_link, child L_M_TIB_link, origin xyz=0.032 0 0 rpy=0 0 0, axis 0 1 0, limit lower=-1.0 upper=1.0 effort=1000.0 velocity=0.5
- added joint R_B_TIB_joint: type revolute, parent R_B_FEM_link, child R_B_TIB_link, origin xyz=-0.027712 0 0 rpy=0 0 0, axis 0 1 0, limit lower=-1.0 upper=1.0 effort=1000.0 velocity=0.5
- added joint R_F_TIB_joint: type revolute, parent R_F_FEM_link, child R_F_TIB_link, origin xyz=-0.027712 0 0 rpy=0 0 0, axis 0 1 0, limit lower=-1.0 upper=1.0 effort=1000.0 velocity=0.5
- added joint R_M_TIB_joint: type revolute, parent R_M_FEM_link, child R_M_TIB_link, origin xyz=-0.032 0 0 rpy=0 0 0, axis 0 1 0, limit lower=-1.0 upper=1.0 effort=1000.0 velocity=0.5
- joint R_B_FEM_joint: origin xyz=-0.014265 -0.010186 0.057284 rpy=0 0 0 -> xyz=-0.007261 0.017438 0.057284 rpy=0 0 0
- joint R_F_FEM_joint: origin xyz=0.001689 -0.017448 0.057284 rpy=0 0 0 -> xyz=-0.007261 -0.017448 0.057284 rpy=0 0 0
- joint R_M_FEM_joint: origin xyz=-0.007261 -0.015954 0.057284 rpy=0 0 0 -> xyz=-0.007261 0.015954 0.057284 rpy=0 0 0

File: urdf/cox.urdf.xacro (robot description, xacro)
@@ -21,16 +21,5 @@
               <material>Gazebo/Green</material>
         </gazebo>
-        <!-- <transmission name="${side}_dock_transmission">
-            <type>transmission_interface/SimpleTransmission</type>
-            <joint name="dock_${side}_joint"> -->
-                <!-- <hardwareInterface>hardware_interface/EffortJointInterface</hardwareInterface> -->
-                <!-- <hardwareInterface>EffortJointInterface</hardwareInterface>
-            </joint>
-            <actuator name="${side}_dock_actuator">
-                <mechanicalReduction>7</mechanicalReduction>
-                <hardwareInterface>EffortJointInterface</hardwareInterface>
-            </actuator>
-        </transmission> -->
     </xacro:macro>
-<!-- ########################## END DOCK GENERATOR ############################ -->
+<!-- ########################## END COXA GENERATOR ############################ -->
 </robot>

File: urdf/tibia.urdf.xacro (robot description, xacro)
@@ -21,16 +21,4 @@
               <material>Gazebo/Green</material>
         </gazebo>
-        <!-- <transmission name="${side}_dock_transmission">
-            <type>transmission_interface/SimpleTransmission</type>
-            <joint name="dock_${side}_joint"> -->
-                <!-- <hardwareInterface>hardware_interface/EffortJointInterface</hardwareInterface> -->
-                <!-- <hardwareInterface>EffortJointInterface</hardwareInterface>
-            </joint>
-            <actuator name="${side}_dock_actuator">
-                <mechanicalReduction>7</mechanicalReduction>
-                <hardwareInterface>EffortJointInterface</hardwareInterface>
-            </actuator>
-        </transmission> -->
     </xacro:macro>
-<!-- ########################## END DOCK GENERATOR ############################ -->
 </robot>

Commit message: feat: add macro for inserting intertias from yaml file

File: robots/hexapod.urdf (robot description, URDF)
Before this commit: robot hexapod, 20 links, 19 joints
Links:
- link L_B_COX_link: mass 0.1 -> 0.02769
- link L_B_FEM_link: mass 0.1 -> 0.02769
- link L_B_TIB_link: mass 0.1 -> 0.02769
- link L_F_COX_link: mass 0.1 -> 0.02769
- link L_F_FEM_link: mass 0.1 -> 0.02769
- link L_F_TIB_link: mass 0.1 -> 0.02769
- link L_M_COX_link: mass 0.1 -> 0.02769
- link L_M_FEM_link: mass 0.1 -> 0.02769
- link L_M_TIB_link: mass 0.1 -> 0.02769
- link R_B_COX_link: mass 0.1 -> 0.02769
- link R_B_FEM_link: mass 0.1 -> 0.02769
- link R_B_TIB_link: mass 0.1 -> 0.02769
- link R_F_COX_link: mass 0.1 -> 0.02769
- link R_F_FEM_link: mass 0.1 -> 0.02769
- link R_F_TIB_link: mass 0.1 -> 0.02769
- link R_M_COX_link: mass 0.1 -> 0.02769
- link R_M_FEM_link: mass 0.1 -> 0.02769
- link R_M_TIB_link: mass 0.1 -> 0.02769

File: robots/hexapod.urdf.xacro (robot description, xacro)
@@ -4,4 +4,7 @@
     <xacro:include filename="$(find hexapod)/urdf/body.urdf.xacro"/>
     <xacro:include filename="$(find hexapod)/urdf/leg.urdf.xacro"/>
+    <xacro:property name="package" value="$(find hexapod)"/>
+    <xacro:property name="origins" value="${load_yaml(package + '/config/joint_origins.yaml')}"/>
+    <xacro:property name="inertias" value="${load_yaml(package + '/config/inertias.yaml')}"/>
     <!-- <xacro:include filename="$(find hexapod)/urdf/hexapod.gazebo" /> -->
     <!-- Footprint link -->

File: urdf/cox.urdf.xacro (robot description, xacro)
@@ -3,5 +3,6 @@
 <!-- ########################## HEXAPOD COXA GENERATOR ############################ -->
     <xacro:macro name="generate_cox" params="side position joint_type:=COX">
-        <xacro:generate_IdOr_link_same_mesh link_name="${side}_${position}_COX_link" stl="coxa_${side}_${position}"/>
+        <!-- <xacro:generate_IdOr_link_same_mesh link_name="${side}_${position}_COX_link" stl="coxa_${side}_${position}"/> -->
+        <xacro:generate_IdOr_SidePosJtype_same_mesh side="${side}" position="${position}" joint_type="COX" stl="coxa_${side}_${position}"/>
         <xacro:property name="coords" value="${origins[side][position][joint_type]}"/>
         <joint name="${side}_${position}_COX_joint" type="revolute" >

File: urdf/femur.urdf.xacro (robot description, xacro)
@@ -3,5 +3,6 @@
 <!-- ########################## HEXAPOD FEMUR GENERATOR ############################ -->
     <xacro:macro name="generate_femur" params="side position joint_type:=FEM">
-        <xacro:generate_IdOr_link_same_mesh link_name="${side}_${position}_FEM_link" stl="femur_${side}_${position}"/>
+        <!-- <xacro:generate_IdOr_link_same_mesh link_name="${side}_${position}_FEM_link" stl="femur_${side}_${position}"/> -->
+        <xacro:generate_IdOr_SidePosJtype_same_mesh side="${side}" position="${position}" joint_type="FEM" stl="femur_${side}_${position}"/>
         <xacro:property name="coords" value="${origins[side][position][joint_type]}"/>
         <joint name="${side}_${position}_FEM_joint" type="revolute" >

File: urdf/general.urdf.xacro (robot description, xacro)
@@ -49,7 +49,7 @@
         </link>
     </xacro:macro>
-    <!--########################## GENERATE IDENTITY ORIGIN LINK WITH IDENTICAL COLLISION/VISUAL MESH XACRO ##########################-->
-    <!-- <xacro:macro name="generate_joint" params="joint_name parent child ">
-        <link name="${link_name}">
+<!--########################## GENERATE HEXAPOD IDENTITY ORIGIN LINK WITH IDENTICAL COLLISION/VISUAL MESH XACRO ##########################-->
+    <xacro:macro name="generate_IdOr_SidePosJtype_same_mesh" params="side:=^|'' position joint_type:=^|'' stl">
+        <link name="${side}_${position}_${joint_type}_link">
             <collision>
                 <xacro:add_stl scale="${SCALE}" fname="${stl}"/>
@@ -58,7 +58,16 @@
                 <xacro:add_stl scale="${SCALE}" fname="${stl}"/>
             </visual>
-            <xacro:MINIMUM_INERTIAL/>
+            <xacro:generate_inertia side="${side}" position="${position}" joint_type="COX"/>
         </link>
-    </xacro:macro> -->
+    </xacro:macro>
+<!--########################## GENERATE IDENTITY ORIGIN IDENTICAL COLLISION/VISUAL MESH XACRO ##########################-->
+    <xacro:macro name="generate_IdOr_CollViz_mesh" params="stl">
+            <collision>
+                <xacro:add_stl scale="${SCALE}" fname="${stl}"/>
+            </collision>
+            <visual>
+                <xacro:add_stl scale="${SCALE}" fname="${stl}"/>
+            </visual>
+    </xacro:macro>
 <!--########################## STL XACRO ##########################-->
     <xacro:macro name="add_stl" params="scale fname">
@@ -105,4 +114,15 @@
         </gazebo>
     </xacro:macro>
+<!-- ########################## HEXAPOD INERTIA GENERATOR ############################ -->
+    <xacro:macro name="generate_inertia" params="side position joint_type">
+        <xacro:property name="coords" value="${origins[side][position][joint_type]}"/>
+        <inertial>
+            <!-- <origin xyz="0 0 0" rpy="0 0 0" /> -->
+            <mass value="${inertias[side][position][joint_type]['m']}"/>
+            <inertia ixx="${inertias[side][position][joint_type]['ixx']}" ixy="${inertias[side][position][joint_type]['ixy']}" ixz="${inertias[side][position][joint_type]['ixz']}"
+            iyy="${inertias[side][position][joint_type]['iyy']}" iyz="${inertias[side][position][joint_type]['iyz']}" izz="${inertias[side][position][joint_type]['izz']}"/>
+        </inertial>
+    </xacro:macro>
+<!-- ########################## END INERTIA GENERATOR ############################ -->
 <!-- ################################################################## -->
 <!-- ############################ COLORS ############################## -->

File: urdf/joint_origins.urdf.xacro (robot description, xacro)
@@ -1,24 +1,4 @@
 <?xml version="1.0"?>
 <robot xmlns:xacro="http://www.ros.org/wiki/xacro">
-<xacro:property name="package" value="$(find hexapod)"/>
-<xacro:property name="origins" value="${load_yaml(package + '/config/joint_origins.yaml')}"/>
-<!-- <xacro:macro name="L_F_COX_ORIG"><origin xyz="0.057077	-0.066312	0.007" rpy="0 0 0"/></xacro:macro>
-<xacro:macro name="L_F_FEM_ORIG"><origin xyz="0.055388	-0.08376	0.064284" rpy="0 0 0"/></xacro:macro>
-<xacro:macro name="L_F_TIB_ORIG"><origin xyz="0.0831	-0.09976	0.064284" rpy="0 0 0"/></xacro:macro>
-<xacro:macro name="L_M_COX_ORIG"><origin xyz="0.0635	0	0.007" rpy="0 0 0"/></xacro:macro>
-<xacro:macro name="L_M_FEM_ORIG"><origin xyz="0.070761	-0.015954	0.064284" rpy="0 0 0"/></xacro:macro>
-<xacro:macro name="L_M_TIB_ORIG"><origin xyz="0.102761	-0.015955	0.064284" rpy="0 0 0"/></xacro:macro>
-<xacro:macro name="L_B_COX_ORIG"><origin xyz="0.057077	0.066312	0.007" rpy="0 0 0"/></xacro:macro>
-<xacro:macro name="L_B_FEM_ORIG"><origin xyz="0.071342	0.056126	0.064284" rpy="0 0 0"/></xacro:macro>
-<xacro:macro name="L_B_TIB_ORIG"><origin xyz="0.099055	0.072126	0.064284" rpy="0 0 0"/></xacro:macro>
-<xacro:macro name="R_F_COX_ORIG"><origin xyz="-0.057077	-0.066312	0.007" rpy="0 0 0"/></xacro:macro>
-<xacro:macro name="R_F_FEM_ORIG"><origin xyz="-0.055388	-0.08376	0.064284" rpy="0 0 0"/></xacro:macro>
-<xacro:macro name="R_F_TIB_ORIG"><origin xyz="-0.0831	-0.09976	0.064284" rpy="0 0 0"/></xacro:macro>
-<xacro:macro name="R_M_COX_ORIG"><origin xyz="-0.0635	0	0.007" rpy="0 0 0"/></xacro:macro>
-<xacro:macro name="R_M_FEM_ORIG"><origin xyz="-0.070761	-0.015954	0.064284" rpy="0 0 0"/></xacro:macro>
-<xacro:macro name="R_M_TIB_ORIG"><origin xyz="-0.102761	-0.015955	0.064284" rpy="0 0 0"/></xacro:macro>
-<xacro:macro name="R_B_COX_ORIG"><origin xyz="-0.057077	0.066312	0.007" rpy="0 0 0"/></xacro:macro>
-<xacro:macro name="R_B_FEM_ORIG"><origin xyz="-0.071342	0.056126	0.064284" rpy="0 0 0"/></xacro:macro>
-<xacro:macro name="R_B_TIB_ORIG"><origin xyz="-0.099055	0.072126	0.06428" rpy="0 0 0"/></xacro:macro> -->
 <!-- <xacro:macro name="get_origin" params="side position joint_type"> -->
     <!-- <xacro:property name="coords" value="${origins['${side}_${position}_${joint_type}']}"/> -->

File: urdf/tibia.urdf.xacro (robot description, xacro)
@@ -4,4 +4,5 @@
     <xacro:macro name="generate_tibia" params="side position joint_type:=TIB">
         <xacro:generate_IdOr_link_same_mesh link_name="${side}_${position}_TIB_link" stl="tibia_${side}_${position}"/>
+        <xacro:generate_IdOr_SidePosJtype_same_mesh side="${side}" position="${position}" joint_type="TIB" stl="tibia_${side}_${position}"/>
         <xacro:property name="coords" value="${origins[side][position][joint_type]}"/>
         <joint name="${side}_${position}_TIB_joint" type="revolute" >
