Commit message: refactor: comment out unused joint origin macros

File: urdf/joint_origins.urdf.xacro (robot description, xacro)
@@ -1,5 +1,7 @@
 <?xml version="1.0"?>
 <robot xmlns:xacro="http://www.ros.org/wiki/xacro">
-<xacro:macro name="L_F_COX_ORIG"><origin xyz="0.057077	-0.066312	0.007" rpy="0 0 0"/></xacro:macro>
+<xacro:property name="package" value="$(find hexapod)"/>
+<xacro:property name="origins" value="${load_yaml(package + '/config/joint_origins.yaml')}"/>
+<!-- <xacro:macro name="L_F_COX_ORIG"><origin xyz="0.057077	-0.066312	0.007" rpy="0 0 0"/></xacro:macro>
 <xacro:macro name="L_F_FEM_ORIG"><origin xyz="0.055388	-0.08376	0.064284" rpy="0 0 0"/></xacro:macro>
 <xacro:macro name="L_F_TIB_ORIG"><origin xyz="0.0831	-0.09976	0.064284" rpy="0 0 0"/></xacro:macro>
@@ -18,7 +20,5 @@
 <xacro:macro name="R_B_COX_ORIG"><origin xyz="-0.057077	0.066312	0.007" rpy="0 0 0"/></xacro:macro>
 <xacro:macro name="R_B_FEM_ORIG"><origin xyz="-0.071342	0.056126	0.064284" rpy="0 0 0"/></xacro:macro>
-<xacro:macro name="R_B_TIB_ORIG"><origin xyz="-0.099055	0.072126	0.06428" rpy="0 0 0"/></xacro:macro>
-<xacro:property name="package" value="$(find hexapod)"/>
-<xacro:property name="origins" value="${load_yaml(package + '/config/joint_origins.yaml')}"/>
+<xacro:macro name="R_B_TIB_ORIG"><origin xyz="-0.099055	0.072126	0.06428" rpy="0 0 0"/></xacro:macro> -->
 <!-- <xacro:macro name="get_origin" params="side position joint_type"> -->
     <!-- <xacro:property name="coords" value="${origins['${side}_${position}_${joint_type}']}"/> -->
