Commit message: feat: move around stuff in tibia.urdf.xacro. There was some copy-pasting and things need to be deleted. Committing before removing entirely.

File: urdf/cox.urdf.xacro (robot description, xacro)
@@ -1,7 +1,7 @@
 <?xml version="1.0"?>
 <robot xmlns:xacro="http://www.ros.org/wiki/xacro">
-<!-- ########################## HEXAPOD TROCOX GENERATOR ############################ -->
+<!-- ########################## HEXAPOD COXA GENERATOR ############################ -->
     <xacro:macro name="generate_cox" params="side position joint_type:=COX">
-        <xacro:generate_IdOr_link_same_mesh link_name="${side}_${position}_COX_link" stl="coxa_2_wheels_${position}_fo"/>
+        <xacro:generate_IdOr_link_same_mesh link_name="${side}_${position}_COX_link" stl="coxa_${position}"/>
         <xacro:property name="coords" value="${origins[side][position][joint_type]}"/>
         <joint name="${side}_${position}_COX_joint" type="revolute" >

File: urdf/femur.urdf.xacro (robot description, xacro)
@@ -3,5 +3,5 @@
 <!-- ########################## HEXAPOD FEMUR GENERATOR ############################ -->
     <xacro:macro name="generate_femur" params="side position joint_type:=FEM">
-        <xacro:generate_IdOr_link_same_mesh link_name="${side}_${position}_FEM_link" stl="femur_no_wheel_${position}_fo"/>
+        <xacro:generate_IdOr_link_same_mesh link_name="${side}_${position}_FEM_link" stl="femur_${position}"/>
         <xacro:property name="coords" value="${origins[side][position][joint_type]}"/>
         <joint name="${side}_${position}_FEM_joint" type="revolute" >

File: urdf/leg.urdf.xacro (robot description, xacro)
@@ -10,4 +10,5 @@
         <xacro:generate_cox side="${side}" position="${position}"/>
         <xacro:generate_femur side="${side}" position="${position}"/>
+        <!-- <xacro:generate_tibia side="left"/> -->
         <xacro:generate_tibia side="${side}" position="${position}"/>
     </xacro:macro>

File: urdf/tibia.urdf.xacro (robot description, xacro)
@@ -1,33 +1,40 @@
 <?xml version="1.0"?>
 <robot xmlns:xacro="http://www.ros.org/wiki/xacro">
-    <!-- <xacro:property name="DOCK_MASS" value="0.01"/> -->
-    <!-- <xacro:property name="FEM_WJ_X" value="-0.070807"/>
-    <xacro:property name="FEM_WJ_Y" value="0.02"/>
-    <xacro:property name="FEM_WJ_Z" value="0.064307"/> -->
-    <!-- FROM ORIGIN -->
-    <!-- <xacro:macro name="FEM_MOTOR_WHEEL_JOINT_ORIGIN">
-        <origin xyz="${FEM_WJ_X} ${FEM_WJ_Y} ${FEM_WJ_Z}" rpy="${PI_2} ${PI} 0" />
-    </xacro:macro> -->
-    <xacro:property name="FEM_WJ_FEM_OFFSET_X" value="0.032"/>
-    <xacro:property name="FEM_WJ_FEM_OFFSET_Y" value="0.004"/>
-    <xacro:property name="FEM_WJ_FEM_OFFSET_Z" value="0.0"/>
-    <!-- FROM TROCOX JOINT -->
-    <xacro:macro name="FEM_MOTOR_WHEEL_JOINT_ORIGIN_FEM_OFFSET">
-        <origin xyz="${FEM_WJ_FEM_OFFSET_X} ${FEM_WJ_FEM_OFFSET_Y} ${FEM_WJ_FEM_OFFSET_Z} " rpy="0 0 0" />
+<!-- ########################## HEXAPOD TIBIA GENERATOR ############################ -->
+    <xacro:macro name="generate_tibia" params="side position joint_type:=TIB">
+        <xacro:generate_IdOr_link_same_mesh link_name="${side}_${position}_COX_link" stl="coxa_${position}"/>
+        <xacro:property name="coords" value="${origins[side][position][joint_type]}"/>
+        <joint name="${side}_${position}_COX_joint" type="revolute" >
+            <origin xyz="${coords['x']} ${coords['y']} ${coords['z']}" rpy="0 0 0"/>
+            <parent link="${side}_${position}_COX_link"/>
+            <!-- NO CHILD LINK <child link="${side}_${position}_COX_link"/> -->
+            <axis xyz="0 1 0" rpy="0 0 0"/>
+            <!-- <limit upper="${PI}" lower="${PI}" effort="10000" velocity="1000"/> -->
+            <limit upper="1.0" lower="-1.0" effort="1000.0" velocity="0.5"/>
+            <!-- <joint_properties damping="1.0" friction="1.0"/> -->
+        </joint>
+         <gazebo reference="${side}_${position}_TIB_link">
+             <mu1 value="${HEX_MU1}"/>
+             <mu2 value="${HEX_MU2}"/>
+             <kp value="${HEX_KP}"/>
+             <kd value="${HEX_KD}"/>
+              <material>Gazebo/Green</material>
+        </gazebo>
+        <!-- <transmission name="${side}_dock_transmission">
+            <type>transmission_interface/SimpleTransmission</type>
+            <joint name="dock_${side}_joint"> -->
+                <!-- <hardwareInterface>hardware_interface/EffortJointInterface</hardwareInterface> -->
+                <!-- <hardwareInterface>EffortJointInterface</hardwareInterface>
+            </joint>
+            <actuator name="${side}_dock_actuator">
+                <mechanicalReduction>7</mechanicalReduction>
+                <hardwareInterface>EffortJointInterface</hardwareInterface>
+            </actuator>
+        </transmission> -->
     </xacro:macro>
-    <!-- <xacro:property name="TIB_FEM_OFFSET_X" value="0.0"/>
-    <xacro:property name="TIB_FEM_OFFSET_Y" value="-0.017845"/>
-    <xacro:property name="TIB_FEM_OFFSET_Z" value="-0.020626"/> -->
-<!-- 001743 -->
-    <xacro:property name="TIB_FEM_OFFSET_X" value="0.0"/>
-    <xacro:property name="TIB_FEM_OFFSET_Y" value="-0.019924"/>
-    <xacro:property name="TIB_FEM_OFFSET_Z" value="-0.01826"/>
-    <!-- FROM TROCOX JOINT -->
-    <xacro:macro name="TIBIA_JOINT_ORIGIN_FEM_OFFSET">
-        <origin xyz="${TIB_FEM_OFFSET_X} ${TIB_FEM_OFFSET_Y} ${TIB_FEM_OFFSET_Z}" rpy="0 0 -${PI}" />
-    </xacro:macro>
-<!-- ########################## HEXAPOD TIBIA GENERATOR ############################ -->
-    <xacro:macro name="generate_tibia" params="side">
-<!-- ########################## FEM WHEEL ############################ -->
+<!-- ########################## END DOCK GENERATOR ############################ -->
+</robot>
+<!-- Moved down. Pretty sure this was copy pasted from docking.
+    ########################## FEM WHEEL ############################
         <link name="tib_motor_wheel_link">
             <xacro:FEM_MOTOR_WHEEL_JOINT_ORIGIN_FEM_OFFSET/>
@@ -79,16 +86,29 @@
               <material>Gazebo/Blue</material>
         </gazebo>
-        <!-- <transmission name="${side}_dock_transmission">
-            <type>transmission_interface/SimpleTransmission</type>
-            <joint name="dock_${side}_joint"> -->
-                <!-- <hardwareInterface>hardware_interface/EffortJointInterface</hardwareInterface> -->
-                <!-- <hardwareInterface>EffortJointInterface</hardwareInterface>
-            </joint>
-            <actuator name="${side}_dock_actuator">
-                <mechanicalReduction>7</mechanicalReduction>
-                <hardwareInterface>EffortJointInterface</hardwareInterface>
-            </actuator>
-        </transmission> -->
+    <!-- <xacro:property name="DOCK_MASS" value="0.01"/> -->
+    <!-- <xacro:property name="FEM_WJ_X" value="-0.070807"/>
+    <xacro:property name="FEM_WJ_Y" value="0.02"/>
+    <xacro:property name="FEM_WJ_Z" value="0.064307"/> -->
+    <!-- FROM ORIGIN -->
+    <!-- <xacro:macro name="FEM_MOTOR_WHEEL_JOINT_ORIGIN">
+        <origin xyz="${FEM_WJ_X} ${FEM_WJ_Y} ${FEM_WJ_Z}" rpy="${PI_2} ${PI} 0" />
+    </xacro:macro> -->
+    <xacro:property name="FEM_WJ_FEM_OFFSET_X" value="0.032"/>
+    <xacro:property name="FEM_WJ_FEM_OFFSET_Y" value="0.004"/>
+    <xacro:property name="FEM_WJ_FEM_OFFSET_Z" value="0.0"/>
+    <!-- FROM TROCOX JOINT -->
+    <xacro:macro name="FEM_MOTOR_WHEEL_JOINT_ORIGIN_FEM_OFFSET">
+        <origin xyz="${FEM_WJ_FEM_OFFSET_X} ${FEM_WJ_FEM_OFFSET_Y} ${FEM_WJ_FEM_OFFSET_Z} " rpy="0 0 0" />
     </xacro:macro>
-<!-- ########################## END DOCK GENERATOR ############################ -->
-</robot>
+    <!-- <xacro:property name="TIB_FEM_OFFSET_X" value="0.0"/>
+    <xacro:property name="TIB_FEM_OFFSET_Y" value="-0.017845"/>
+    <xacro:property name="TIB_FEM_OFFSET_Z" value="-0.020626"/> -->
+<!-- 001743 -->
+    <xacro:property name="TIB_FEM_OFFSET_X" value="0.0"/>
+    <xacro:property name="TIB_FEM_OFFSET_Y" value="-0.019924"/>
+    <xacro:property name="TIB_FEM_OFFSET_Z" value="-0.01826"/>
+    <!-- FROM TROCOX JOINT -->
+    <xacro:macro name="TIBIA_JOINT_ORIGIN_FEM_OFFSET">
+        <origin xyz="${TIB_FEM_OFFSET_X} ${TIB_FEM_OFFSET_Y} ${TIB_FEM_OFFSET_Z}" rpy="0 0 -${PI}" />
+    </xacro:macro>
+-->
