Commit message: feat: add more info to poses.txt, reformat, and begin work on urdf inertial.

File: urdf/body.urdf.xacro (robot description, xacro)
@@ -1,5 +1,5 @@
 <?xml version="1.0"?>
 <robot xmlns:xacro="http://www.ros.org/wiki/xacro">
-    <xacro:property name="HEX_MASS" value="0.1"/>
+    <xacro:property name="HEX_MASS" value="0.1"/> <!--body mass: 1.503462, Total Mass: 2.812273-->
     <xacro:property name="HEX_LENGTH" value="0.4"/>
     <xacro:property name="HEX_WIDTH" value="0.05"/>
